Commit message: urdf edit

File: urdf/turtlebot3_burger_leader.gazebo.xacro (robot description, xacro)
@@ -26,13 +26,4 @@
     <fdir1>1 0 0</fdir1>
     <material>Gazebo/FlatBlack</material>
-  </gazebo>
-  <gazebo reference="Apriltag36_11_00000">
-    <material>
-      <script>
-        <uri>model://Apriltag36_11_00000/materials/scripts</uri>
-        <uri>model://Apriltag36_11_00000/materials/textures</uri>
-        <name>Apriltag36_11_00000</name>
-      </script>
-    </material>
   </gazebo>
   <gazebo reference="caster_back_link">
@@ -167,3 +158,12 @@
     </sensor>
   </gazebo>
+  <gazebo reference="Apriltag36_11_00000">
+    <material>
+      <script>
+        <uri>model://Apriltag36_11_00000/materials/scripts</uri>
+        <uri>model://Apriltag36_11_00000/materials/textures</uri>
+        <name>Apriltag36_11_00000</name>
+      </script>
+    </material>
+  </gazebo>
 </robot>

File: urdf/turtlebot3_burger_leader.urdf.xacro (robot description, xacro)
@@ -166,5 +166,5 @@
   <link name="camera_rgb_optical_frame"/>
   <joint name="tag_joint" type="fixed">
-    <parent link="base_link"/>
+    <parent link="base_scan"/>
     <child link="Apriltag36_11_00000"/>
     <origin xyz="0 0 0.28" rpy="0 0 0"/>

Commit message: simulation leader bot

File: urdf/turtlebot3_burger_leader.gazebo.xacro (robot description, xacro)
@@ -26,13 +26,4 @@
     <fdir1>1 0 0</fdir1>
     <material>Gazebo/FlatBlack</material>
-  </gazebo>
-  <gazebo reference="Apriltag36_11_00000">
-    <material>
-      <script>
-        <uri>model://Apriltag36_11_00000/materials/scripts</uri>
-        <uri>model://Apriltag36_11_00000/materials/textures</uri>
-        <name>Apriltag36_11_00000</name>
-      </script>
-    </material>
   </gazebo>
   <gazebo reference="caster_back_link">
@@ -167,3 +158,6 @@
     </sensor>
   </gazebo>
+ <gazebo reference="Apriltag36_11_00000_link">
+    <material>Apriltag36_11_00000</material>
+  </gazebo>
 </robot>

File: urdf/turtlebot3_burger_leader.urdf.xacro (robot description, xacro)
@@ -2,5 +2,8 @@
 <robot name="turtlebot3_burger" xmlns:xacro="http://ros.org/wiki/xacro">
   <xacro:include filename="$(find turtlebot3_description)/urdf/common_properties.xacro"/>
-  <xacro:include filename="$(find turtlebot3_description)/urdf/turtlebot3_burger.gazebo.xacro"/>
+  <xacro:include filename="$(find aue_finals)/urdf/turtlebot3_burger_leader.gazebo.xacro"/>
+  <material name="Apriltag36_11_00000">
+    <texture filename="package://aue_finals/models/Apriltag36_11_00000/materials/textures/Apriltag36_11_00000.png"/>
+  </material>
   <link name="base_footprint"/>
   <joint name="base_joint" type="fixed">
@@ -124,5 +127,4 @@
         <mesh filename="package://turtlebot3_description/meshes/sensors/lds.stl" scale="0.001 0.001 0.001"/>
       </geometry>
-      <material name="dark"/>
     </visual>
     <collision>
@@ -167,12 +169,12 @@
   <joint name="tag_joint" type="fixed">
     <parent link="base_link"/>
-    <child link="Apriltag36_11_00000"/>
-    <origin xyz="0 0 0.28" rpy="0 0 0"/>
+    <child link="Apriltag36_11_00000_link"/>
+    <origin xyz="-0.1 0 0.1" rpy="0 0 0"/>
   </joint>
-  <link name="Apriltag36_11_00000">
+  <link name="Apriltag36_11_00000_link">
     <visual>
       <origin xyz="0 0 0" rpy="1.57 0 0"/>
       <geometry>
-        <box size="0.010 0.100 0.100"/>
+        <box size="0.001 0.200 0.200"/>
       </geometry>
     </visual>
