Commit message: Final codes as used in demo, cleaned up

File: urdf/turtlebot3_burger_leader.urdf.xacro (robot description, xacro)
@@ -170,5 +170,5 @@
     <parent link="base_link"/>
     <child link="Apriltag36_11_00000_link"/>
-    <origin xyz="-0.1 0 0.1" rpy="0 0 0"/>
+    <origin xyz="-0.12 0 0.1" rpy="0 0 0"/>
   </joint>
   <link name="Apriltag36_11_00000_link">
